File: projects/ring/ring.kicad_pcb (KiCad board)
At the start: 4 copper layers, 12 x 20 mm, 38 parts, among them Q1 AOCA32116E, U1 STM32WB55CEU6TR, U2 LSM6DSO32TR, U3 ANT016008LCS2442MA2, U4 BQ297xy, U5 TPS62840DLCR, Y1 NX1612SA-32.000MHZ-CHP-CIS-3

Commit message: just shipped first rev :fingers_crossed:
Parts:
- added C7: C_100pF, Capacitor_SMD:C_0201_0603Metric, F.Cu at (72.5, 24.1)
- C2: footprint Capacitor_SMD:C_0402_1005Metric -> Capacitor_SMD:C_0201_0603Metric
- moved C2 0.31 mm to (71.9, 23.8)
Routing:
- net /TPS_STOP: track 12.4 -> 13.5 mm
- net GND: track 15.1 -> 16.2 mm, vias 45 -> 46
